File: dmx-cover/dmx-cover.kicad_pcb (KiCad board)
At the start: 2 copper layers, 66 x 18 mm, 7 parts

Commit message: Update to KiCad 7.0
Parts:
- H1: value MountingHole -> MountingHole_1mm; footprint V2_Mechanical:Mounting_Hole_1 -> V2_Mechanical:MountingHole_1mm
- H2, H3: value MountingHole_Pad -> MountingHole_2mm_Pad_5.2mm; footprint V2_Mechanical:Mounting_Hole_Pad_2-5.2 -> V2_Mechanical:Mounting_Hole_2mm_Pad_5.2mm
Connections:
- net /SHIELD renamed GND
