File: dmx.kicad_pcb (KiCad board)
At the start: 4 copper layers, 66 x 18 mm, 41 parts, among them J101 SJ2-25504B-SMT-TR, J102 CORTEX-DEBUG, J103 JAE_DX07S016JA1R1500, SW101 SW_Push, SW102 SW_Push, U101 LTC2851xDD, U102 ATSAMD51G, U103 AP2112K-3.3, Y101 32.768kHz

Commit message: Update to KiCad 7.0
Parts:
- removed C105, C112: 100n, Capacitor_SMD:C_0603_1608Metric
- removed J101: SJ2-25504B-SMT-TR, V2_Connector_Audio:CUI_SJ2-25504B-SMT-TR
- removed U103: AP2112K-3.3, Package_TO_SOT_SMD:SOT-23-5
- added C201: 0u1, Capacitor_SMD:C_0603_1608Metric, F.Cu at (164.8, 98.8)
- added J201: SJ2-25504B-SMT-TR, V2_Connector_Audio:CUI_SJ2-25504B-SMT-TR, F.Cu at (177.8, 106.0)
- added U201: LTC2863, V2_Package_DFN_QFN:DFN-8-1EP_3x3mm_P0.5mm_EP1.65x2.38mm, F.Cu at (164.8, 101.5)
- C104, C106, C107, C108, C109, C113: value 100n -> 0u1
- J103: value JAE_DX07S016JA1R1500 -> JAE_DX07S016JA3; footprint V2_Connector_USB:JAE_DX07S016JA1R1500 -> V2_Connector_USB:JAE_DX07S016JA3
- SPACER101, SPACER102: value 977?2434030 -> 9774030243
- U101: value LTC2851xDD -> TPS78433QWDRBRQ1; footprint Package_DFN_QFN:DFN-8-1EP_3x3mm_P0.5mm_EP1.66x2.38mm -> V2_Package_SON:VSON-8-1_3x3mm_P0.65_EP1.65x2.4mm
- Y101: value 32.768kHz -> 32k768
- moved U101 34.0 mm to (135.0, 111.2), turned to 180 degrees
- moved C110 3.76 mm to (138.0, 111.2), turned to 90 degrees
- moved C111 1.52 mm to (132.0, 111.2), turned to 90 degrees
Connections:
- C106 pad 1: +3.3V -> +3V3
- C107 pad 1: +3.3V -> +3V3
- C108 pad 1: +3.3V -> +3V3
- C109 pad 1: +3.3V -> +3V3
- C110 pad 1: +3.3V -> +3V3
- J102 pad 1: +3.3V -> +3V3
- R101 pad 1: +3.3V -> +3V3
- U101 pad 1: +5V -> +3V3
- U101 pad 3: /DMX -> unconnected-(U101-Pad3)
- U101 pad 4: GND -> unconnected-(U101-Pad4)
- U101 pad 5: Net-(J101-Pad3) -> GND
- U101 pad 6: Net-(J101-Pad5) -> unconnected-(U101-Pad6)
- U101 pad 7: unconnected-(U101-Pad7) -> +5V
- U101 pad 8: unconnected-(U101-Pad8) -> +5V
- U102 pad 17: +3.3V -> +3V3
- U102 pad 31: /DMX -> /DMX-Data
- U102 pad 36: +3.3V -> +3V3
- U102 pad 4: +3.3V -> +3V3
- U102 pad 44: +3.3V -> +3V3
- U102 pad 6: +3.3V -> +3V3
Routing:
- net /DMX: track 29.2 -> 0.00 mm
- net +3V3: track 0.00 -> 18.7 mm, vias 0 -> 9
- net +3.3V: track 17.9 -> 0.00 mm, vias 10 -> 0
- net /DMX-Data: track 0.00 -> 17.6 mm
- net Net-(J101-Pad3): track 14.2 -> 0.00 mm
- net Net-(J201-R1): track 0.00 -> 13.1 mm
- net Net-(J101-Pad5): track 11.5 -> 0.00 mm
- net GND: track 38.5 -> 29.2 mm, vias 38 -> 36
- net Net-(U201-Z): track 0.00 -> 7.78 mm
- net +5V: track 14.8 -> 19.8 mm, vias 12 -> 10
- net /Button: track 26.3 -> 27.2 mm
- added copper zone on In2.Cu, net +3V3
- removed copper zone on In2.Cu, net +3.3V
